File: schematics/BlueRetro3V3/BlueRetro3V3.kicad_sch (KiCad schematic)
At the start: 23 parts, among them J1 Conn_01x04, J2 Conn_01x04, J3 Conn_01x02, Q1 2N7000, Q2 2N7000, SW1 BOOT, SW2 RESET, U1 ESP32 MH-ET Live D1 mini

Commit message: schematics minor update
Other:
- note added: "Boot Button"
- moved on the sheet: D4, D5, Q1, Q2, R1, R4, R5
